Commit message: Update a1.urdf

File: resources/robots/a1/urdf/a1.urdf (robot description, URDF)
Before this commit: robot a1_description, 23 links, 22 joints
Links:
- added link ejt, mass 0.001; visual box size=0.001 0.001 0.001
Joints:
- added joint ejt_joint: type fixed, parent trunk, child ejt, origin xyz=0 0 0 rpy=0 0 0

Commit message: Update a1.urdf

File: resources/robots/a1/urdf/a1.urdf (robot description, URDF)
Before this commit: robot a1_description, 24 links, 23 joints
Joints:
- joint FL_calf_joint: origin xyz=0 0 -0.2 rpy=0 0 0 -> xyz=0 0 -0.2 rpy=0 -1.2 0
- joint FL_hip_joint: origin xyz=0.183 0.047 0 rpy=0 0 0 -> xyz=0.183 0.047 0 rpy=0 0.1 0
- joint FL_thigh_joint: origin xyz=0 0.08505 0 rpy=0 0 0 -> xyz=0 0.08505 0 rpy=0 1.0 0
- joint FR_calf_joint: origin xyz=0 0 -0.2 rpy=0 0 0 -> xyz=0 0 -0.2 rpy=0 -1.2 0
- joint FR_hip_joint: origin xyz=0.183 -0.047 0 rpy=0 0 0 -> xyz=0.183 -0.047 0 rpy=0 -0.1 0
- joint FR_thigh_joint: origin xyz=0 -0.08505 0 rpy=0 0 0 -> xyz=0 -0.08505 0 rpy=0 1.0 0
- joint RL_calf_joint: origin xyz=0 0 -0.2 rpy=0 0 0 -> xyz=0 0 -0.2 rpy=0 -1.2 0
- joint RL_hip_joint: origin xyz=-0.183 0.047 0 rpy=0 0 0 -> xyz=-0.183 0.047 0 rpy=0 0.1 0
- joint RL_thigh_joint: origin xyz=0 0.08505 0 rpy=0 0 0 -> xyz=0 0.08505 0 rpy=0 1.0 0
- joint RR_calf_joint: origin xyz=0 0 -0.2 rpy=0 0 0 -> xyz=0 0 -0.2 rpy=0 -1.2 0
- joint RR_hip_joint: origin xyz=-0.183 -0.047 0 rpy=0 0 0 -> xyz=-0.183 -0.047 0 rpy=0 -0.1 0
- joint RR_thigh_joint: origin xyz=0 -0.08505 0 rpy=0 0 0 -> xyz=0 -0.08505 0 rpy=0 1.0 0
